File: esp8266-12-breakout.kicad_pcb (KiCad board)
At the start: 2 copper layers, 32.4 x 38.7 mm, 13 parts, among them P1 ftdi, P2 CONN_01X14, SW1 SW_PUSH, U1 AP1117D33

Commit message: fixed gpio 4/5 mixup
Parts:
- R3: value 120r -> 68r
Connections:
- P2 pad 5: /gpio5 -> /gpio4
- P2 pad 6: /gpio4 -> /gpio5
- esp8266 pad 13: /gpio4 -> /gpio5
- esp8266 pad 14: /gpio5 -> /gpio4
Routing:
- net /gpio5: track 22.1 -> 19.7 mm
- net /gpio4: track 19.7 -> 22.1 mm
Changed lines of the file:
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@@
     (links 38)
     (no_connects 0)
-    (area 109.804999 95.83 143.387572 140.635001)
+    (area 109.804999 101.549999 142.290001 140.385001)
     (thickness 1.6)
     (drawings 619)
@@
       (net 3 +3V3))
     (pad 5 thru_hole oval (at 0 -10.16 180) (size 2.032 1.7272) (drill 1.016) (layers *.Cu *.Mask B.SilkS)
+      (net 10 /gpio4))
+    (pad 6 thru_hole oval (at 0 -12.7 180) (size 2.032 1.7272) (drill 1.016) (layers *.Cu *.Mask B.SilkS)
       (net 9 /gpio5))
-    (pad 6 thru_hole oval (at 0 -12.7 180) (size 2.032 1.7272) (drill 1.016) (layers *.Cu *.Mask B.SilkS)
-      (net 10 /gpio4))
     (pad 7 thru_hole oval (at 0 -15.24 180) (size 2.032 1.7272) (drill 1.016) (layers *.Cu *.Mask B.SilkS)
       (net 5 /gpio0))
@@
       (net 5 /gpio0))
     (pad 13 smd oval (at 8 15.9) (size 1.524 3) (layers F.Cu F.Paste F.Mask)
+      (net 9 /gpio5))
+    (pad 14 smd oval (at 10 15.9) (size 1.524 3) (layers F.Cu F.Paste F.Mask)
       (net 10 /gpio4))
-    (pad 14 smd oval (at 10 15.9) (size 1.524 3) (layers F.Cu F.Paste F.Mask)
-      (net 9 /gpio5))
     (pad 15 smd oval (at 12 15.9) (size 1.524 3) (layers F.Cu F.Paste F.Mask)
       (net 7 /rx))
@@
       (effects (font (size 1 1) (thickness 0.15)))
     )
-    (fp_text value 120r (at 0 2.3 180) (layer F.Fab)
+    (fp_text value 68r (at 0 2.3 180) (layer F.Fab)
       (effects (font (size 1 1) (thickness 0.15)))
     )
@@
   )
   (gr_line (start 113.705 109) (end 113.705 104) (layer F.SilkS) (width 0.2))
-  (gr_text gnd (at 133.604 139.192 360) (layer F.SilkS)
+  (gr_text gnd (at 133.604 139.192) (layer F.SilkS)
     (effects (font (size 1 1) (thickness 0.2)) (justify left))
   )
@@
     (effects (font (size 1 1) (thickness 0.2)) (justify left))
   )
-  (gr_text 5v (at 113.5 110 360) (layer F.SilkS)
+  (gr_text 5v (at 113.5 110) (layer F.SilkS)
     (effects (font (size 1 1) (thickness 0.2)) (justify left))
   )
-  (gr_text 3.3v (at 113.5 113 360) (layer F.SilkS)
+  (gr_text 3.3v (at 113.5 113) (layer F.SilkS)
     (effects (font (size 1 1) (thickness 0.2)) (justify left))
   )
-  (gr_text 05 (at 114.5 115.824) (layer F.SilkS)
+  (gr_text 04 (at 114.3 115.824) (layer F.SilkS)
     (effects (font (size 1 1) (thickness 0.2)) (justify left))
   )
-  (gr_text 04 (at 114.3 118.11) (layer F.SilkS)
+  (gr_text 05 (at 114.3 118.11) (layer F.SilkS)
     (effects (font (size 1 1) (thickness 0.2)) (justify left))
   )
@@
   (segment (start 130.248121 131.338877) (end 130.248121 133.657879) (width 0.25) (layer F.Cu) (net 8))
   (via (at 129.667 134.239) (size 0.6) (drill 0.4) (layers F.Cu B.Cu) (net 8))
-  (segment (start 124.443306 123.513306) (end 124.390696 123.513306) (width 0.25) (layer F.Cu) (net 9))
-  (segment (start 128.714 127.784) (end 124.443306 123.513306) (width 0.25) (layer F.Cu) (net 9))
-  (segment (start 116.44739 115.57) (end 124.090697 123.213307) (width 0.25) (layer B.Cu) (net 9))
-  (segment (start 128.714 128.522) (end 128.714 127.784) (width 0.25) (layer F.Cu) (net 9))
-  (segment (start 124.090697 123.213307) (end 124.390696 123.513306) (width 0.25) (layer B.Cu) (net 9))
-  (segment (start 112.395 115.57) (end 116.44739 115.57) (width 0.25) (layer B.Cu) (net 9))
-  (via (at 124.390696 123.513306) (size 0.6) (drill 0.4) (layers F.Cu B.Cu) (net 9))
-  (segment (start 124.021 124.079) (end 123.995264 124.079) (width 0.25) (layer F.Cu) (net 10))
-  (segment (start 126.714 126.772) (end 124.021 124.079) (width 0.25) (layer F.Cu) (net 10))
-  (segment (start 123.995264 124.079) (end 123.571 124.079) (width 0.25) (layer F.Cu) (net 10))
-  (segment (start 123.271001 123.779001) (end 123.571 124.079) (width 0.25) (layer B.Cu) (net 10))
-  (segment (start 112.395 118.11) (end 117.602 118.11) (width 0.25) (layer B.Cu) (net 10))
-  (segment (start 117.602 118.11) (end 123.271001 123.779001) (width 0.25) (layer B.Cu) (net 10))
-  (segment (start 126.714 128.522) (end 126.714 126.772) (width 0.25) (layer F.Cu) (net 10))
-  (via (at 123.571 124.079) (size 0.6) (drill 0.4) (layers F.Cu B.Cu) (net 10))
+  (segment (start 117.602 118.11) (end 123.271001 123.779001) (width 0.25) (layer B.Cu) (net 9))
+  (segment (start 112.395 118.11) (end 117.602 118.11) (width 0.25) (layer B.Cu) (net 9))
+  (segment (start 124.021 124.079) (end 123.995264 124.079) (width 0.25) (layer F.Cu) (net 9))
+  (segment (start 126.714 126.772) (end 124.021 124.079) (width 0.25) (layer F.Cu) (net 9))
+  (segment (start 123.995264 124.079) (end 123.571 124.079) (width 0.25) (layer F.Cu) (net 9))
+  (segment (start 123.271001 123.779001) (end 123.571 124.079) (width 0.25) (layer B.Cu) (net 9))
+  (segment (start 126.714 128.522) (end 126.714 126.772) (width 0.25) (layer F.Cu) (net 9))
+  (via (at 123.571 124.079) (size 0.6) (drill 0.4) (layers F.Cu B.Cu) (net 9))
+  (segment (start 124.443306 123.513306) (end 124.390696 123.513306) (width 0.25) (layer F.Cu) (net 10))
+  (segment (start 128.714 127.784) (end 124.443306 123.513306) (width 0.25) (layer F.Cu) (net 10))
+  (segment (start 116.44739 115.57) (end 124.090697 123.213307) (width 0.25) (layer B.Cu) (net 10))
+  (segment (start 128.714 128.522) (end 128.714 127.784) (width 0.25) (layer F.Cu) (net 10))
+  (segment (start 124.090697 123.213307) (end 124.390696 123.513306) (width 0.25) (layer B.Cu) (net 10))
+  (segment (start 112.395 115.57) (end 116.44739 115.57) (width 0.25) (layer B.Cu) (net 10))
+  (via (at 124.390696 123.513306) (size 0.6) (drill 0.4) (layers F.Cu B.Cu) (net 10))
   (segment (start 113.661 123.19) (end 112.395 123.19) (width 0.25) (layer B.Cu) (net 11))
   (segment (start 116.985775 123.19) (end 113.661 123.19) (width 0.25) (layer B.Cu) (net 11))

Commit message: added reset pin to breakout for deepsleep
Connections:
- P2 pad 2: GND -> +5V
- P2 pad 3: +5V -> +3V3
- P2 pad 4: +3V3 -> /reset
Routing:
- net /reset: track 35.8 -> 59.8 mm, vias 0 -> 1
- net GND: track 63.8 -> 61.2 mm
- net +3V3: track 104.8 -> 105.6 mm
Other:
- board text added: "3.3v ftdi"
- board text added: "rst"
Changed lines of the file:
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@@
     (area 109.804999 101.549999 142.290001 140.385001)
     (thickness 1.6)
-    (drawings 619)
-    (tracks 210)
+    (drawings 621)
+    (tracks 216)
     (zones 0)
     (modules 13)
@@
     (descr "Through hole pin header")
     (tags "pin header")
-    (fp_text reference P1 (at 2.286 4.826 540) (layer F.SilkS)
+    (fp_text reference P1 (at -2.286 12.7 540) (layer F.SilkS)
       (effects (font (size 1 1) (thickness 0.15)))
     )
@@
       (net 1 GND))
     (pad 2 thru_hole oval (at 0 -2.54 180) (size 2.032 1.7272) (drill 1.016) (layers *.Cu *.Mask B.SilkS)
-      (net 1 GND))
+      (net 2 +5V))
     (pad 3 thru_hole oval (at 0 -5.08 180) (size 2.032 1.7272) (drill 1.016) (layers *.Cu *.Mask B.SilkS)
-      (net 2 +5V))
+      (net 3 +3V3))
     (pad 4 thru_hole oval (at 0 -7.62 180) (size 2.032 1.7272) (drill 1.016) (layers *.Cu *.Mask B.SilkS)
-      (net 3 +3V3))
+      (net 6 /reset))
     (pad 5 thru_hole oval (at 0 -10.16 180) (size 2.032 1.7272) (drill 1.016) (layers *.Cu *.Mask B.SilkS)
       (net 10 /gpio4))
@@
     (pad 2 smd rect (at 2.9 0.00232 270) (size 2.18 1.6) (layers F.Cu F.Paste F.Mask)
       (net 1 GND))
+  )
+  (gr_text "3.3v ftdi" (at 125.476 139.192) (layer F.SilkS)
+    (effects (font (size 1 1) (thickness 0.2)))
+  )
+  (gr_text rst (at 114.046 112.776) (layer F.SilkS)
+    (effects (font (size 1 1) (thickness 0.2)) (justify left))
   )
   (gr_line (start 113.705 113.915) (end 116.705 113.915) (layer F.SilkS) (width 0.2))
@@
     (effects (font (size 1 1) (thickness 0.2)) (justify left))
   )
-  (gr_text gnd (at 114.5 105 270) (layer F.SilkS)
-    (effects (font (size 1 1) (thickness 0.2)) (justify left))
-  )
-  (gr_text 5v (at 113.5 110) (layer F.SilkS)
-    (effects (font (size 1 1) (thickness 0.2)) (justify left))
-  )
-  (gr_text 3.3v (at 113.5 113) (layer F.SilkS)
+  (gr_text gnd (at 114.808 104.14 270) (layer F.SilkS)
+    (effects (font (size 1 1) (thickness 0.2)) (justify left))
+  )
+  (gr_text 5v (at 114.046 108.204) (layer F.SilkS)
+    (effects (font (size 1 1) (thickness 0.2)) (justify left))
+  )
+  (gr_text 3.3v (at 114.046 110.49) (layer F.SilkS)
     (effects (font (size 1 1) (thickness 0.2)) (justify left))
   )
@@
   (segment (start 121.785 103.005) (end 120.777 104.013) (width 0.5) (layer F.Cu) (net 1))
   (segment (start 120.777 104.013) (end 120.269 104.013) (width 0.5) (layer F.Cu) (net 1))
-  (segment (start 112.395 107.95) (end 112.395 105.41) (width 0.5) (layer F.Cu) (net 1))
   (segment (start 120.269 104.013) (end 117.54104 104.013) (width 0.5) (layer F.Cu) (net 1))
   (segment (start 117.54104 104.013) (end 117.094 104.46004) (width 0.5) (layer F.Cu) (net 1))
   (segment (start 117.094 104.46004) (end 113.34496 104.46004) (width 0.5) (layer F.Cu) (net 1))
   (segment (start 113.34496 104.46004) (end 112.395 105.41) (width 0.5) (layer F.Cu) (net 1))
-  (segment (start 117.094 108.458) (end 114.427 108.458) (width 0.5) (layer F.Cu) (net 2))
-  (segment (start 114.427 108.458) (end 113.911 108.974) (width 0.5) (layer F.Cu) (net 2))
-  (segment (start 113.911 108.974) (end 113.911 109.1264) (width 0.5) (layer F.Cu) (net 2))
-  (segment (start 112.5474 110.49) (end 112.395 110.49) (width 0.5) (layer F.Cu) (net 2))
-  (segment (start 113.911 109.1264) (end 112.5474 110.49) (width 0.5) (layer F.Cu) (net 2))
+  (segment (start 112.395 107.95) (end 116.586 107.95) (width 0.5) (layer F.Cu) (net 2))
+  (segment (start 116.586 107.95) (end 117.094 108.458) (width 0.5) (layer F.Cu) (net 2))
+  (segment (start 112.903 108.458) (end 112.395 107.95) (width 0.5) (layer F.Cu) (net 2))
   (segment (start 120.269 108.585) (end 117.221 108.585) (width 0.5) (layer F.Cu) (net 2))
   (segment (start 117.221 108.585) (end 117.094 108.458) (width 0.5) (layer F.Cu) (net 2))
+  (segment (start 112.395 110.49) (end 113.911 110.49) (width 0.5) (layer F.Cu) (net 3))
+  (segment (start 113.911 110.49) (end 115.943 112.522) (width 0.5) (layer F.Cu) (net 3))
+  (segment (start 115.943 112.522) (end 117.452 112.522) (width 0.5) (layer F.Cu) (net 3))
+  (segment (start 117.452 112.522) (end 118.714 112.522) (width 0.5) (layer F.Cu) (net 3))
+  (segment (start 112.5474 110.49) (end 112.395 110.49) (width 0.5) (layer F.Cu) (net 3))
   (segment (start 131.30761 138.57201) (end 129.794 137.0584) (width 0.5) (layer B.Cu) (net 3))
   (segment (start 136.779 138.050602) (end 136.257592 138.57201) (width 0.5) (layer B.Cu) (net 3))
@@
   (segment (start 128.714 112.522) (end 128.714 111.784) (width 0.5) (layer F.Cu) (net 3))
   (segment (start 126.543001 109.613001) (end 121.935001 109.613001) (width 0.5) (layer F.Cu) (net 3))
-  (segment (start 118.714 112.522) (end 112.903 112.522) (width 0.5) (layer F.Cu) (net 3))
-  (segment (start 112.903 112.522) (end 112.395 113.03) (width 0.5) (layer F.Cu) (net 3))
   (segment (start 120.269 106.299) (end 121.785 106.299) (width 0.5) (layer F.Cu) (net 3))
   (segment (start 121.785 106.299) (end 121.935001 106.449001) (width 0.5) (layer F.Cu) (net 3))
@@
   (segment (start 124.714 126.328998) (end 124.714 126.772) (width 0.25) (layer F.Cu) (net 5))
   (segment (start 124.714 126.772) (end 124.714 128.522) (width 0.25) (layer F.Cu) (net 5))
+  (segment (start 131.699 115.189) (end 132.714 114.174) (width 0.25) (layer F.Cu) (net 6))
+  (segment (start 132.714 114.174) (end 132.714 112.522) (width 0.25) (layer F.Cu) (net 6))
+  (segment (start 112.395 113.03) (end 129.54 113.03) (width 0.25) (layer B.Cu) (net 6))
+  (segment (start 129.54 113.03) (end 131.699 115.189) (width 0.25) (layer B.Cu) (net 6))
+  (via (at 131.699 115.189) (size 0.6) (drill 0.4) (layers F.Cu B.Cu) (net 6))
+  (segment (start 112.903 112.522) (end 112.395 113.03) (width 0.5) (layer F.Cu) (net 6))
   (segment (start 132.714 112.522) (end 132.714 112.797264) (width 0.25) (layer F.Cu) (net 6))
   (segment (start 123.084597 121.733989) (end 119.754237 125.064349) (width 0.25) (layer F.Cu) (net 6))

Commit message: serial silk screen and v2
Parts:
- moved R3 6.86 mm to (138.4, 104.6)
- moved D1 6.75 mm to (138.4, 107.2)
- moved C2 5.09 mm to (130.8, 106.2)
- moved C3 4.58 mm to (134.1, 106.2)
Routing:
- net GND: track 61.2 -> 57.7 mm
- net +3V3: track 105.6 -> 103.1 mm
- net Net-(D1-Pad1): track 3.35 -> 2.55 mm
Other:
- board text added: "3.3v serial usb cable"
- board text added: "dtr rx tx vcc cts gnd"
- board text added: "esp8266-12 v2 breakout board Matt Venn 2015"
- board text removed: "3.3v ftdi"
- board text removed: "esp8266-12 breakout board Matt Venn 2015"

Commit message: swapped gpio 4&5
Connections:
- P2 pad 5: /gpio4 -> /gpio5
- P2 pad 6: /gpio5 -> /gpio4
- esp8266 pad 13: /gpio5 -> /gpio4
- esp8266 pad 14: /gpio4 -> /gpio5
Routing:
- net /gpio5: track 19.7 -> 22.1 mm
- net /gpio4: track 22.1 -> 19.7 mm
Changed lines of the file:
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@@
     (links 38)
     (no_connects 0)
-    (area 109.804999 95.83 142.290001 140.635001)
+    (area 109.804999 101.549999 142.290001 140.385001)
     (thickness 1.6)
     (drawings 621)
@@
     (pad_to_mask_clearance 0)
     (aux_axis_origin 109.855 101.473)
-    (grid_origin 52.705 145.415)
+    (grid_origin 110.109 101.6)
     (visible_elements FFFEFF7F)
     (pcbplotparams
@@
       (net 6 /reset))
     (pad 5 thru_hole oval (at 0 -10.16 180) (size 2.032 1.7272) (drill 1.016) (layers *.Cu *.Mask B.SilkS)
+      (net 9 /gpio5))
+    (pad 6 thru_hole oval (at 0 -12.7 180) (size 2.032 1.7272) (drill 1.016) (layers *.Cu *.Mask B.SilkS)
       (net 10 /gpio4))
-    (pad 6 thru_hole oval (at 0 -12.7 180) (size 2.032 1.7272) (drill 1.016) (layers *.Cu *.Mask B.SilkS)
-      (net 9 /gpio5))
     (pad 7 thru_hole oval (at 0 -15.24 180) (size 2.032 1.7272) (drill 1.016) (layers *.Cu *.Mask B.SilkS)
       (net 5 /gpio0))
@@
       (net 5 /gpio0))
     (pad 13 smd oval (at 8 15.9) (size 1.524 3) (layers F.Cu F.Paste F.Mask)
+      (net 10 /gpio4))
+    (pad 14 smd oval (at 10 15.9) (size 1.524 3) (layers F.Cu F.Paste F.Mask)
       (net 9 /gpio5))
-    (pad 14 smd oval (at 10 15.9) (size 1.524 3) (layers F.Cu F.Paste F.Mask)
-      (net 10 /gpio4))
     (pad 15 smd oval (at 12 15.9) (size 1.524 3) (layers F.Cu F.Paste F.Mask)
       (net 7 /rx))
@@
     (effects (font (size 1 1) (thickness 0.2)) (justify left))
   )
-  (gr_text 04 (at 114.3 115.5954) (layer F.SilkS)
+  (gr_text 05 (at 114.3 115.5954) (layer F.SilkS)
     (effects (font (size 1 1) (thickness 0.2)) (justify left))
   )
-  (gr_text 05 (at 114.3 118.11) (layer F.SilkS)
+  (gr_text 04 (at 114.3 118.11) (layer F.SilkS)
     (effects (font (size 1 1) (thickness 0.2)) (justify left))
   )
@@
   (segment (start 130.248121 131.338877) (end 130.248121 133.657879) (width 0.25) (layer F.Cu) (net 8))
   (via (at 129.667 134.239) (size 0.6) (drill 0.4) (layers F.Cu B.Cu) (net 8))
-  (segment (start 117.602 118.11) (end 123.271001 123.779001) (width 0.25) (layer B.Cu) (net 9))
-  (segment (start 112.395 118.11) (end 117.602 118.11) (width 0.25) (layer B.Cu) (net 9))
-  (segment (start 124.021 124.079) (end 123.995264 124.079) (width 0.25) (layer F.Cu) (net 9))
-  (segment (start 126.714 126.772) (end 124.021 124.079) (width 0.25) (layer F.Cu) (net 9))
-  (segment (start 123.995264 124.079) (end 123.571 124.079) (width 0.25) (layer F.Cu) (net 9))
-  (segment (start 123.271001 123.779001) (end 123.571 124.079) (width 0.25) (layer B.Cu) (net 9))
-  (segment (start 126.714 128.522) (end 126.714 126.772) (width 0.25) (layer F.Cu) (net 9))
-  (via (at 123.571 124.079) (size 0.6) (drill 0.4) (layers F.Cu B.Cu) (net 9))
-  (segment (start 124.443306 123.513306) (end 124.390696 123.513306) (width 0.25) (layer F.Cu) (net 10))
-  (segment (start 128.714 127.784) (end 124.443306 123.513306) (width 0.25) (layer F.Cu) (net 10))
-  (segment (start 116.44739 115.57) (end 124.090697 123.213307) (width 0.25) (layer B.Cu) (net 10))
-  (segment (start 128.714 128.522) (end 128.714 127.784) (width 0.25) (layer F.Cu) (net 10))
-  (segment (start 124.090697 123.213307) (end 124.390696 123.513306) (width 0.25) (layer B.Cu) (net 10))
-  (segment (start 112.395 115.57) (end 116.44739 115.57) (width 0.25) (layer B.Cu) (net 10))
-  (via (at 124.390696 123.513306) (size 0.6) (drill 0.4) (layers F.Cu B.Cu) (net 10))
+  (segment (start 124.443306 123.513306) (end 124.390696 123.513306) (width 0.25) (layer F.Cu) (net 9))
+  (segment (start 128.714 127.784) (end 124.443306 123.513306) (width 0.25) (layer F.Cu) (net 9))
+  (segment (start 116.44739 115.57) (end 124.090697 123.213307) (width 0.25) (layer B.Cu) (net 9))
+  (segment (start 128.714 128.522) (end 128.714 127.784) (width 0.25) (layer F.Cu) (net 9))
+  (segment (start 124.090697 123.213307) (end 124.390696 123.513306) (width 0.25) (layer B.Cu) (net 9))
+  (segment (start 112.395 115.57) (end 116.44739 115.57) (width 0.25) (layer B.Cu) (net 9))
+  (via (at 124.390696 123.513306) (size 0.6) (drill 0.4) (layers F.Cu B.Cu) (net 9))
+  (segment (start 117.602 118.11) (end 123.271001 123.779001) (width 0.25) (layer B.Cu) (net 10))
+  (segment (start 112.395 118.11) (end 117.602 118.11) (width 0.25) (layer B.Cu) (net 10))
+  (segment (start 124.021 124.079) (end 123.995264 124.079) (width 0.25) (layer F.Cu) (net 10))
+  (segment (start 126.714 126.772) (end 124.021 124.079) (width 0.25) (layer F.Cu) (net 10))
+  (segment (start 123.995264 124.079) (end 123.571 124.079) (width 0.25) (layer F.Cu) (net 10))
+  (segment (start 123.271001 123.779001) (end 123.571 124.079) (width 0.25) (layer B.Cu) (net 10))
+  (segment (start 126.714 128.522) (end 126.714 126.772) (width 0.25) (layer F.Cu) (net 10))
+  (via (at 123.571 124.079) (size 0.6) (drill 0.4) (layers F.Cu B.Cu) (net 10))
   (segment (start 113.661 123.19) (end 112.395 123.19) (width 0.25) (layer B.Cu) (net 11))
   (segment (start 116.985775 123.19) (end 113.661 123.19) (width 0.25) (layer B.Cu) (net 11))
